File: h/h.kicad_pcb (KiCad board)
At the start: 2 copper layers, 37.9 x 69.1 mm, 35 parts, among them J1 USB_C_Receptacle_USB2.0, M1 Motor_DC, Q1 Q_NMOS_GDS, SW1 SW_L, SW2 SW_UP, SW3 SW_C, SW4 SW_DW, SW5 SW_R, U1 ESP32-S3-DEVKITC-1U-N8R8, U2 MCP73831-2-OT

Commit message: check desc
add code file and organize rest for main firmware
and completed assembly
Routing:
- net GND: track 369.7 -> 302.6 mm
- net SW_DW: track 0.00 -> 23.1 mm
- net SW_C: track 0.00 -> 14.3 mm
- net SW_UP: track 0.00 -> 13.5 mm
- net SW_L: track 0.00 -> 11.1 mm
- net Net-(L2-Pad1): track 16.4 -> 9.64 mm
- net Net-(L2-Pad2): track 0.00 -> 6.72 mm
- net SW_R: track 0.00 -> 5.14 mm
